Commit message: fully configured-ish

File: src/klaw_description/urdf/klaw.xacro (robot description, xacro)
@@ -1,7 +1,9 @@
 <?xml version="1.0" ?>
 <robot name="klaw" xmlns:xacro="http://www.ros.org/wiki/xacro">
-<xacro:include filename="$(find klaw_description)/urdf/materials.xacro" />
-<xacro:include filename="$(find klaw_description)/urdf/welder.trans" />
-<xacro:include filename="$(find klaw_description)/urdf/welder.gazebo" />
+<xacro:include filename="$(find klaw_description)/urdf/klaw.trans" />
+<xacro:include filename="$(find klaw_description)/urdf/klaw.gazebo" />
+<xacro:include filename="$(find klaw_description)/urdf/ros2_control.xacro" />
+<link name="world">
+</link>
 <link name="base_link">
   <inertial>
@@ -15,5 +17,4 @@
       <mesh filename="file://$(find klaw_description)/meshes/base_link.stl" scale="0.001 0.001 0.001"/>
     </geometry>
-    <material name="silver"/>
   </visual>
   <collision>
@@ -35,5 +36,4 @@
       <mesh filename="file://$(find klaw_description)/meshes/link_1_1.stl" scale="0.001 0.001 0.001"/>
     </geometry>
-    <material name="silver"/>
   </visual>
   <collision>
@@ -55,5 +55,4 @@
       <mesh filename="file://$(find klaw_description)/meshes/link_2_1.stl" scale="0.001 0.001 0.001"/>
     </geometry>
-    <material name="silver"/>
   </visual>
   <collision>
@@ -75,5 +74,4 @@
       <mesh filename="file://$(find klaw_description)/meshes/link_3_1.stl" scale="0.001 0.001 0.001"/>
     </geometry>
-    <material name="silver"/>
   </visual>
   <collision>
@@ -95,5 +93,4 @@
       <mesh filename="file://$(find klaw_description)/meshes/link_4_1.stl" scale="0.001 0.001 0.001"/>
     </geometry>
-    <material name="silver"/>
   </visual>
   <collision>
@@ -115,5 +112,4 @@
       <mesh filename="file://$(find klaw_description)/meshes/link_5_1.stl" scale="0.001 0.001 0.001"/>
     </geometry>
-    <material name="silver"/>
   </visual>
   <collision>
@@ -135,5 +131,4 @@
       <mesh filename="file://$(find klaw_description)/meshes/gripper_1.stl" scale="0.001 0.001 0.001"/>
     </geometry>
-    <material name="silver"/>
   </visual>
   <collision>
@@ -155,5 +150,4 @@
       <mesh filename="file://$(find klaw_description)/meshes/klaw_1_1.stl" scale="0.001 0.001 0.001"/>
     </geometry>
-    <material name="silver"/>
   </visual>
   <collision>
@@ -175,5 +169,4 @@
       <mesh filename="file://$(find klaw_description)/meshes/klaw_2_1.stl" scale="0.001 0.001 0.001"/>
     </geometry>
-    <material name="silver"/>
   </visual>
   <collision>
@@ -184,4 +177,8 @@
   </collision>
 </link>
+<joint name="world_joint" type="fixed">
+  <parent link="world"/>
+  <child link="base_link"/>
+</joint>
 <joint name="joint_1" type="continuous">
   <origin xyz="0.0 0.0 0.175" rpy="0 0 0"/>
@@ -228,9 +225,10 @@
 </joint>
 <joint name="gripper_2" type="revolute">
-  <origin xyz="0.215 0.13 0.0" rpy="0 0 0"/>
+  <origin xyz="0.215 0.13 0.0" rpy="6.283185 0 0"/>
   <parent link="gripper"/>
   <child link="klaw_2_1"/>
   <axis xyz="0.0 0.0 -1.0"/>
-  <limit upper="6.283185" lower="3.228859" effort="100" velocity="100"/>
+  <!-- <limit upper="6.283185" lower="3.228859" effort="100" velocity="100"/> -->
+  <limit upper="0" lower="-3.228859" effort="100" velocity="100"/>
 </joint>
 </robot>

Commit message: some minor changes

File: src/klaw_description/urdf/klaw.xacro (robot description, xacro)
@@ -178,4 +178,5 @@
 </link>
 <joint name="world_joint" type="fixed">
+  <origin xyz="0.0 0.0 0.55" rpy="0 0 0"/>
   <parent link="world"/>
   <child link="base_link"/>

Commit message: Two positions thus far

File: src/klaw_description/urdf/klaw.xacro (robot description, xacro)
@@ -178,5 +178,5 @@
 </link>
 <joint name="world_joint" type="fixed">
-  <origin xyz="0.0 0.0 0.55" rpy="0 0 0"/>
+  <origin xyz="0.0 0.0 0.0" rpy="0 0 0"/>
   <parent link="world"/>
   <child link="base_link"/>
